File: TayType_IMUbreakout/TapType_IMUbreakout/TapType_IMUbreakout.kicad_sch (KiCad schematic)
At the start: 7 parts, among them J1 Conn_01x06, U1 LSM6DS3

Commit message: Update IMU breakout files
Parts:
- added D2, D3: SMF5.0A, Diode_SMD:D_SOD-123, symbol SMF5.0A:SMF5.0A
- C1, C2: footprint (none) -> Capacitor_SMD:C_0603_1608Metric_Pad1.08x0.95mm_HandSolder
- D1: footprint (none) -> LED_SMD:LED_0603_1608Metric_Pad1.05x0.95mm_HandSolder
- J1: footprint (none) -> FPC-SMD_6P-P0.50_FPC-05FB-6PH20:FPC-SMD_6P-P0.50_FPC-05FB-6PH20
- R1, R4: footprint (none) -> Resistor_SMD:R_0603_1608Metric_Pad0.98x0.95mm_HandSolder
Connections:
- net +3.3V: now also J1.6 (Pin_6); no longer J1.1 (Pin_1)
- net GND: now also J1.2 (Pin_2), D2.A, D3.A; no longer J1.5 (Pin_5)
- net INT1: now also J1.1 (Pin_1), D3.C; no longer J1.6 (Pin_6)
- net SA0: now also J1.3 (Pin_3), D2.C; no longer J1.4 (Pin_4)
- net SCL: now also J1.4 (Pin_4); no longer J1.3 (Pin_3)
- net SDA: now also J1.5 (Pin_5); no longer J1.2 (Pin_2)
Other:
- moved on the sheet: C1, C2, D1, J1, R1
